Commit message: fea: final lidar and ir sensors

File: src/myrobot/myrobot_description/urdf/macro.xacro (robot description, xacro)
@@ -18,7 +18,7 @@
   </xacro:macro>
   <!-- WHEEL MACRO -->
-  <xacro:macro name="wheel" params="wheel_prefix parent_link left_right radius width *joint_origin">
+  <xacro:macro name="wheel" params="wheel_prefix parent_link left_right radius mass width *joint_origin">
     <link name="${wheel_prefix}_wheel">
-      <xacro:cylinder_inertial length="${width}" mass="${wheel_mass}" radius="${radius}">
+      <xacro:cylinder_inertial length="${width}" mass="${mass}" radius="${radius}">
         <origin rpy="${PI/2} 0 0" xyz="0 0 0"/>
       </xacro:cylinder_inertial>
@@ -51,4 +51,29 @@
       </joint>
     </transmission>
+  </xacro:macro>
+  <!-- LIDAR MACRO -->
+  <xacro:macro name="lidar" params="lidar_prefix parent_link radius mass width">
+    <joint name="${lidar_prefix}_lidar_joint" type="fixed">
+        <parent link="${parent_link}"/>
+        <child link="${lidar_prefix}_lidar_frame"/>
+        <origin xyz="-0.05 0 0.09" rpy="0 0 0"/>
+    </joint>
+    <link name="${lidar_prefix}_lidar_frame">
+      <xacro:cylinder_inertial length="${width}" mass="${mass}" radius="${radius}">
+        <origin rpy="${PI/2} 0 0" xyz="0 0 0"/>
+      </xacro:cylinder_inertial>
+      <visual>
+        <origin rpy="0 0 0" xyz="0 0 0"/>
+        <geometry>
+          <mesh filename="package://myrobot_description/meshes/rplidar.dae" scale="${radius} ${radius} ${width/2}"/>
+        </geometry>
+      </visual>
+      <collision>
+        <origin rpy="0 0 0" xyz="0 0 0"/>
+        <geometry>
+          <cylinder length="${width}" radius="${radius}"/>
+        </geometry>
+      </collision>
+    </link>
   </xacro:macro>
   <!-- OTHER -->
@@ -86,4 +111,5 @@
     </joint>
   </xacro:macro>
+  <!-- IR-SENSOR MACRO -->
   <xacro:macro name="ir_sensor" params="name parent sx sy sz *origin">
     <link name="ir_sensor_${name}">
@@ -101,4 +127,32 @@
       <xacro:insert_block name="origin"/>
     </joint>
+    <gazebo reference="ir_sensor_${name}">
+      <sensor type="ray" name="ir_sensor_${name}_ray">
+        <pose>0 0 0 0 0 0</pose>
+        <visualize>true</visualize>
+        <update_rate>50</update_rate>
+        <always_on>true</always_on>
+        <ray>
+          <scan>
+            <horizontal>
+              <samples>1</samples>
+              <resolution>1</resolution>
+              <min_angle>0.0</min_angle>
+              <max_angle>0.0</max_angle>
+            </horizontal>
+          </scan>
+        </ray>
+        <plugin name="ir_sensor_${name}_plugin" filename="libgazebo_ros_range.so">
+          <topicName>/myrobot/sensor/${name}</topicName>
+          <frameName>ir_sensor_${name}</frameName>
+          <gaussianNoise>0.005</gaussianNoise>
+          <alwaysOn>true</alwaysOn>
+          <updateRate>5</updateRate>
+          <visualize>true</visualize>
+          <radiation>infrared</radiation>
+          <fov>0.436</fov>
+        </plugin>
+      </sensor>
+    </gazebo>
   </xacro:macro>
   <xacro:macro name="ir_sensor_rot" params="name parent distance yaw pitch">
@@ -106,5 +160,5 @@
       sx="0.003" sy="0.008" sz="0.008">
       <origin rpy="0 ${pitch} ${yaw}"
-       xyz="${distance*cos(yaw)} ${distance*sin(yaw)} 0"/>
+       xyz="${distance*cos(yaw)} ${distance*sin(yaw)} 0.03"/>
     </xacro:ir_sensor>
   </xacro:macro>

File: src/myrobot/myrobot_description/urdf/myrobot.xacro (robot description, xacro)
@@ -2,9 +2,11 @@
 <robot name="myrobot" xmlns:xacro="http://www.ros.org/wiki/xacro">
   <!-- ============ Enter xacro properties here (if you want) =============== -->
+  <!-- Параметры кузова робота -->
 	<xacro:property name="chassis_width" value="0.05"/>
 	<xacro:property name="chassis_length" value="0.05"/>
 	<xacro:property name="chassis_height" value="0.05"/>
 	<xacro:property name="chassis_z" value="0.05"/>
-	<xacro:property name="chassis_mass" value="2000"/>
+	<xacro:property name="chassis_mass" value="1"/>
+  <!-- Параметры колес робота -->
   <xacro:property name="wheel_radius" value="0.02"/>
   <xacro:property name="wheel_mass" value="0.1"/>
@@ -12,8 +14,13 @@
   <xacro:property name="wheelbase_offset" value="0.07"/>
   <xacro:property name="wheelbase_length" value="0.1"/>
+  <!-- Параметры лидара робота -->
+  <xacro:property name="lidar_radius" value="0.001"/>
+  <xacro:property name="lidar_width" value="0.001"/>
+  <xacro:property name="lidar_mass" value="0.1"/>
   <!-- ============ Including macros and materials =============== -->
-	<xacro:include filename="$(find myrobot_description)/urdf/myrobot.gazebo" />
   <xacro:include filename="$(find myrobot_description)/urdf/macro.xacro"/>
   <xacro:include filename="$(find myrobot_description)/urdf/materials.xacro"/>
+  <!-- Подключаем макросы gazebo для использования макроса rplidar_a2_gpu лидаром -->
+	<xacro:include filename="$(find myrobot_simulator)/urdf/macro.gazebo.xacro" />
   <!-- ============ Some magic. Do not touch =============== -->
   <link name="rs_t265_pose_frame">
@@ -24,5 +31,6 @@
     <child link="base_link"/>
   </joint>
-    <!-- ============ Enter base_link code here =============== -->
+  <!-- ============ Enter base_link code here =============== -->
+  <!-- Описываем линк кузова робота -->
   <link
     name="base_link">
@@ -54,7 +62,7 @@
     </collision>
   </link>
-    <!-- ============ Enter wheels code here =============== -->
-  <!-- Использование макроса колеса -->
-  <xacro:wheel wheel_prefix="right" parent_link="base_link" left_right="1" radius="${wheel_radius}" width="${wheel_width}">
+  <!-- ============ Enter wheels code here =============== -->
+  <!-- Описываем линк правого колеса робота -->
+  <xacro:wheel wheel_prefix="right" parent_link="base_link" left_right="1" radius="${wheel_radius}" mass="${wheel_mass}" width="${wheel_width}">
     <origin xyz=
       "${wheelbase_offset}
@@ -62,5 +70,6 @@
        ${wheel_radius}"/>
   </xacro:wheel>
-  <xacro:wheel wheel_prefix="left" parent_link="base_link" left_right="-1" radius="${wheel_radius}" width="${wheel_width}">
+  <!-- Описываем линк левого колеса робота -->
+  <xacro:wheel wheel_prefix="left" parent_link="base_link" left_right="-1" radius="${wheel_radius}" mass="${wheel_mass}" width="${wheel_width}">
     <origin xyz=
       "${wheelbase_offset}
@@ -68,6 +77,17 @@
        ${wheel_radius}"/>
   </xacro:wheel>
-    <!-- ============ Enter sensors code here =============== -->
-    <!-- ============ LIDAR =============== -->
-    <!-- ============ IR sensors =============== -->
+  <!-- ============ LIDAR =============== -->
+  <!-- Вызываем макросы, необходимые для работы лидара -->
+  <xacro:lidar lidar_prefix="base" parent_link="base_link" radius="${lidar_radius}" mass="${lidar_mass}" width="${lidar_width}"></xacro:lidar>
+  <xacro:rplidar_a2_gpu max_angle="360" min_angle="0" name="base_lidar" ray_count="400" ros_topic="/myrobot/rplidar/scan" update_rate="20"/>
+  <!-- ============ Enter sensors code here =============== -->
+  <!-- ============ IR sensors =============== -->
+  <!-- Описываем передние датчики дистанции робота -->
+  <xacro:ir_sensor_rot name="front_0" parent="base_link" distance="0.135" yaw="0" pitch="0"></xacro:ir_sensor_rot>
+  <xacro:ir_sensor_rot name="front_1" parent="base_link" distance="0.135" yaw="0.4" pitch="0"></xacro:ir_sensor_rot>
+  <xacro:ir_sensor_rot name="front_2" parent="base_link" distance="0.135" yaw="-0.4" pitch="0"></xacro:ir_sensor_rot>
+  <!-- Описываем задние датчики дистанции робота -->
+  <xacro:ir_sensor_rot name="back_0" parent="base_link" distance="-0.175" yaw="0" pitch="3.142"></xacro:ir_sensor_rot>
+  <xacro:ir_sensor_rot name="back_1" parent="base_link" distance="-0.175" yaw="0.3" pitch="3.142"></xacro:ir_sensor_rot>
+  <xacro:ir_sensor_rot name="back_2" parent="base_link" distance="-0.175" yaw="-0.3" pitch="3.142"></xacro:ir_sensor_rot>
 </robot>

File: src/myrobot/myrobot_simulator/urdf/macro.gazebo.xacro (robot description, xacro)
@@ -101,3 +101,15 @@
     <frameName>ir_sensor_front_2</frameName>
   </xacro:ir_sensor_gazebo>
+  <xacro:ir_sensor_gazebo name="back_0">
+    <topicName>/myrobot/sensor/back_0</topicName>
+    <frameName>ir_sensor_back_0</frameName>
+  </xacro:ir_sensor_gazebo>
+  <xacro:ir_sensor_gazebo name="back_1">
+    <topicName>/myrobot/sensor/back_1</topicName>
+    <frameName>ir_sensor_back_1</frameName>
+  </xacro:ir_sensor_gazebo>
+  <xacro:ir_sensor_gazebo name="back_2">
+    <topicName>/myrobot/sensor/back_2</topicName>
+    <frameName>ir_sensor_back_2</frameName>
+  </xacro:ir_sensor_gazebo>
 </robot>
