Commit message: fea: keyboard_teleop and auto_teleop for ir sensors

File: src/myrobot/myrobot_description/urdf/myrobot.xacro (robot description, xacro)
@@ -7,8 +7,8 @@
 	<xacro:property name="chassis_height" value="0.05"/>
 	<xacro:property name="chassis_z" value="0.05"/>
-	<xacro:property name="chassis_mass" value="1"/>
+	<xacro:property name="chassis_mass" value="0.01"/>
   <!-- Параметры колес робота -->
   <xacro:property name="wheel_radius" value="0.02"/>
-  <xacro:property name="wheel_mass" value="0.1"/>
+  <xacro:property name="wheel_mass" value="0.001"/>
   <xacro:property name="wheel_width" value="0.02"/>
   <xacro:property name="wheelbase_offset" value="0.07"/>
@@ -17,5 +17,5 @@
   <xacro:property name="lidar_radius" value="0.001"/>
   <xacro:property name="lidar_width" value="0.001"/>
-  <xacro:property name="lidar_mass" value="0.1"/>
+  <xacro:property name="lidar_mass" value="0.0001"/>
   <!-- ============ Including macros and materials =============== -->
   <xacro:include filename="$(find myrobot_description)/urdf/macro.xacro"/>
